File: kicad-teensy-epaper.sch (KiCad schematic (older format))
At the start: 3 parts, among them J1 HEADER-FEMALE-34POS-FFC-SMT-1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

Commit message: start the schematic and layout over
Parts:
- removed J?: HEADER-MALE-25POS-TH-1x25-P0.1IN, Wickerlib:CONN-HEADER-STRAIGHT-P2.54MM-1x25, symbol HEADER-MALE-25POS-TH-1x25-P0.1IN
- removed J?: HEADER-MALE-9POS-TH-1x09-P0.1IN, Wickerlib:CONN-HEADER-STRAIGHT-P2.54MM-1x09, symbol HEADER-MALE-9POS-TH-1x09-P0.1IN
Connections:
- net labels added: NC1
Changed lines of the file:
@@
 EESchema Schematic File Version 2
 LIBS:wickerlib
+LIBS:kicad-teensy-epaper-cache
 EELAYER 25 0
 EELAYER END
@@
 Comment4 ""
 $EndDescr
+Wire Wire Line
+	4975 3725 6125 3725
+Wire Wire Line
+	4975 3625 6125 3625
+Wire Wire Line
+	4975 3525 6125 3525
+Wire Wire Line
+	4975 3425 6125 3425
+Wire Wire Line
+	4975 3325 6125 3325
+Wire Wire Line
+	4975 3225 6125 3225
+Wire Wire Line
+	4975 3125 6125 3125
+Wire Wire Line
+	4975 3025 6125 3025
+Wire Wire Line
+	4975 2925 6125 2925
+Wire Wire Line
+	6125 2825 4975 2825
+Wire Wire Line
+	4975 2725 6125 2725
+Wire Wire Line
+	6125 2625 4975 2625
+Wire Wire Line
+	4975 2525 6125 2525
+Wire Wire Line
+	4975 2425 6125 2425
+Wire Wire Line
+	6125 2325 4975 2325
+Wire Wire Line
+	4975 2225 6125 2225
+Wire Wire Line
+	6125 2125 4975 2125
+Wire Wire Line
+	4975 2025 6125 2025
+Wire Wire Line
+	6125 1925 4975 1925
+Wire Wire Line
+	4975 1825 6125 1825
+Wire Wire Line
+	6125 5125 4975 5125
+Wire Wire Line
+	4975 5025 6125 5025
+Wire Wire Line
+	6125 4925 4975 4925
+Wire Wire Line
+	4975 4825 6125 4825
+Wire Wire Line
+	6125 4725 4975 4725
+Wire Wire Line
+	4975 3825 6125 3825
+Wire Wire Line
+	6125 3925 4975 3925
+Wire Wire Line
+	4975 4025 6125 4025
+Wire Wire Line
+	6125 4125 4975 4125
+Wire Wire Line
+	4975 4225 6125 4225
+Wire Wire Line
+	6125 4325 4975 4325
+Wire Wire Line
+	4975 4425 6125 4425
+Wire Wire Line
+	6125 4525 4975 4525
+Wire Wire Line
+	4975 4625 6125 4625
 $Comp
 L HEADER-FEMALE-34POS-FFC-SMT-1x34-P0.5MM J1
-U 1 1 5870583B
-P 5025 3700
-F 0 "J1" H 4975 4750 50  0000 L CNN
-F 1 "HEADER-FEMALE-34POS-FFC-SMT-1x34-P0.5MM" H 4975 1250 50  0000 L CNN
-F 2 "Wickerlib:CONN-HEADER-FH34SRJ-34S-0.5SH" H 5025 3350 50  0001 C CIN
-F 3 "https://cdn.harwin.com/pdfs/60page140.pd://www.hirose.com/product/en/download_file/key_name/FH34SRJ/category/Catalog/doc_file_id/31646/?file_category_id=4&item_id=27&is_series=1" H 5025 3700 5   0001 C CNN
-F 4 "HEADER FEMALE 34POS SMT 1x34 0.5MMP" H 5025 3350 50  0001 C CIN "Description"
-F 5 "Hirose" H 5025 3350 50  0001 C CIN "MF_Name"
-F 6 "FH34SRJ-34S-0.5SH(99)" H 5025 3350 50  0001 C CIN "MF_PN"
-F 7 "Digikey" H 5025 3350 50  0001 C CIN "S1_Name"
-F 8 "H124726CT-ND" H 5025 3350 50  0001 C CIN "S1_PN"
-	1    5025 3700
-	-1   0    0    1
+U 1 1 58799DE1
+P 6325 2775
+F 0 "J1" H 6275 3825 50  0000 L CNN
+F 1 "HEADER-FEMALE-34POS-FFC-SMT-1x34-P0.5MM" H 6275 325 50  0000 L CNN
+F 2 "Wickerlib:CONN-HEADER-FH34SRJ-34S-0.5SH" H 6325 2425 50  0001 C CIN
+F 3 "https://cdn.harwin.com/pdfs/60page140.pd://www.hirose.com/product/en/download_file/key_name/FH34SRJ/category/Catalog/doc_file_id/31646/?file_category_id=4&item_id=27&is_series=1" H 6325 2775 5   0001 C CNN
+F 4 "HEADER FEMALE 34POS SMT 1x34 0.5MMP" H 6325 2425 50  0001 C CIN "Description"
+F 5 "Hirose" H 6325 2425 50  0001 C CIN "MF_Name"
+F 6 "FH34SRJ-34S-0.5SH(99)" H 6325 2425 50  0001 C CIN "MF_PN"
+F 7 "Digikey" H 6325 2425 50  0001 C CIN "S1_Name"
+F 8 "H124726CT-ND" H 6325 2425 50  0001 C CIN "S1_PN"
+	1    6325 2775
+	1    0    0    -1
 $EndComp
-$Comp
-L HEADER-MALE-25POS-TH-1x25-P0.1IN J?
-U 1 1 58705B9E
-P 6575 3450
-F 0 "J?" H 6525 4750 50  0000 L CNN
-F 1 "HEADER-MALE-25POS-TH-1x25-P0.1IN" H 6525 2150 50  0000 L CNN
-F 2 "Wickerlib:CONN-HEADER-STRAIGHT-P2.54MM-1x25" H 6575 3100 50  0001 C CIN
-F 3 "https://cdn.harwin.com/pdfs/60page140.pdf" H 6575 3450 5   0001 C CNN
-F 4 "HEADER MALE 25POS TH 1x25 0.1”" H 6575 3100 50  0001 C CIN "Description"
-F 5 "Harwin" H 6575 3100 50  0001 C CIN "MF_Name"
-F 6 "M20-9992046" H 6575 3100 50  0001 C CIN "MF_PN"
-F 7 "Digikey" H 6575 3100 50  0001 C CIN "S1_Name"
-F 8 "952-1902-ND" H 6575 3100 50  0001 C CIN "S1_PN"
-	1    6575 3450
-	1    0    0    1
-$EndComp
-Wire Wire Line
-	5225 4650 6375 4650
-Wire Wire Line
-	5225 4550 6375 4550
-Wire Wire Line
-	5225 4450 6375 4450
-Wire Wire Line
-	5225 4350 6375 4350
-Wire Wire Line
-	5225 4250 6375 4250
-Wire Wire Line
-	5225 4150 6375 4150
-Wire Wire Line
-	5225 4050 6375 4050
-Wire Wire Line
-	5225 3950 6375 3950
-Wire Wire Line
-	5225 3850 6375 3850
-Wire Wire Line
-	6375 3750 5225 3750
-Wire Wire Line
-	5225 3650 6375 3650
-Wire Wire Line
-	6375 3550 5225 3550
-Wire Wire Line
-	5225 3450 6375 3450
-Wire Wire Line
-	5225 3350 6375 3350
-Wire Wire Line
-	6375 3250 5225 3250
-Wire Wire Line
-	5225 3150 6375 3150
-Wire Wire Line
-	6375 3050 5225 3050
-Wire Wire Line
-	5225 2950 6375 2950
-Wire Wire Line
-	6375 2850 5225 2850
-Wire Wire Line
-	5225 2750 6375 2750
-Wire Wire Line
-	6375 2650 5225 2650
-Wire Wire Line
-	5225 2550 6375 2550
-Wire Wire Line
-	6375 2450 5225 2450
-Wire Wire Line
-	5225 2350 6375 2350
-Wire Wire Line
-	6375 2250 5225 2250
-$Comp
-L HEADER-MALE-9POS-TH-1x09-P0.1IN J?
-U 1 1 58706087
-P 6575 1750
-F 0 "J?" H 6525 2250 50  0000 L CNN
-F 1 "HEADER-MALE-9POS-TH-1x09-P0.1IN" H 6525 1250 50  0000 L CNN
-F 2 "Wickerlib:CONN-HEADER-STRAIGHT-P2.54MM-1x09" H 6575 1400 50  0001 C CIN
-F 3 "https://cdn.harwin.com/pdfs/60page140.pdf" H 6575 1750 5   0001 C CNN
-F 4 "HEADER MALE 9POS TH 1x09 0.1”" H 6575 1400 50  0001 C CIN "Description"
-F 5 "Harwin" H 6575 1400 50  0001 C CIN "MF_Name"
-F 6 "M20-9992046" H 6575 1400 50  0001 C CIN "MF_PN"
-F 7 "Digikey" H 6575 1400 50  0001 C CIN "S1_Name"
-F 8 "952-1902-ND" H 6575 1400 50  0001 C CIN "S1_PN"
-	1    6575 1750
-	1    0    0    1
-$EndComp
-Wire Wire Line
-	5225 1350 6375 1350
-Wire Wire Line
-	6375 1450 5225 1450
-Wire Wire Line
-	5225 1550 6375 1550
-Wire Wire Line
-	6375 1650 5225 1650
-Wire Wire Line
-	5225 1750 6375 1750
-Wire Wire Line
-	6375 1850 5225 1850
-Wire Wire Line
-	5225 1950 6375 1950
-Wire Wire Line
-	6375 2050 5225 2050
-Wire Wire Line
-	5225 2150 6375 2150
+Text GLabel 4975 1825 0    50   Input ~ 0
+NC1
 $EndSCHEMATC

Commit message: finish redrawing the EAGLE schematic in KiCad
TODO: make sure the correct parts are used for passives and mosfet
Parts:
- added C? (x10): CAP-CER-1UF, Wickerlib:RLC-0603-SMD, symbol CAP-CER-1UF-25V-X7R-0603
- added D? (x3): DIODE, Wickerlib:DIODE-SMA, symbol DIODE-SCHOTTKY-40V-1A-MBRA140-SMA
- added J?: TEENSY-LC, Wickerlib:TEENSY-LC-SILK, symbol TEENSY-LC
- added L?: INDUCTOR, symbol INDUCTOR
- added Q?: MOSFET, Wickerlib:SOT-23-3, symbol MOSFET-N-20V-3.2A-NTR4501NT1G
- added R?: 2.2R 1%, symbol R
Connections:
- net labels added: BS1, BUSY, DOUT, GDR, GND, NC2, NC3, NC4, NC5, NC6, NC7, NC8, PRVGI, PRVGL, RESE, SCK, TSCL, TSDA, VCI?, VCOM, VDD, VDDIO, VGH, VGH2, VGL, VPP, VSH, VSI, VSL, VSS, ^CS, ^D/C, ^RES
- wire segments 34 -> 55
- no-connect marks 0 -> 23
Other:
- moved on the sheet: J1

Commit message: first attempt at layout, 1 air wire remains
Parts:
- removed C? (x2): CAP-CER-1UF, Wickerlib:RLC-0603-SMD, symbol CAP-CER-1UF-25V-X7R-0603
- removed J?: TEENSY-LC, Wickerlib:TEENSY-LC-SILK, symbol TEENSY-LC
- removed Q?: MOSFET, Wickerlib:SOT-23-3, symbol MOSFET-N-20V-3.2A-NTR4501NT1G
- added C10, C3: CAP-CER-1UF, Capacitors_SMD:C_0805_HandSoldering, symbol CAP-CER-1UF-25V-X7R-0603
- added J1: TEENSY3.2-72MHz, Wickerlib:TEENSY-3.2-SILK, symbol TEENSY3.2-72MHz
- added Q1: Q_NMOS_GDS, TO_SOT_Packages_SMD:SOT-23_Handsoldering, symbol Q_NMOS_GDS
- C1, C2, C4, C5, C6, C7, C8, C9: renamed from C?; footprint Wickerlib:RLC-0603-SMD -> Capacitors_SMD:C_0805_HandSoldering
- D1, D2, D3: renamed from D?; footprint Wickerlib:DIODE-SMA -> Diodes_SMD:SOD-123
- L1: renamed from L?; footprint (none) -> Inductors:Inductor_1212
- R1: renamed from R?; footprint (none) -> Resistors_SMD:R_0805_HandSoldering
- renumbered J1 to J2
Connections:
- net labels removed: PRVGI, VCI?, VSI
- wire segments 55 -> 50
- no-connect marks 23 -> 34
Other:
- moved on the sheet: C1, C2, C4, C5, C6, C7, C8, C9, D1, D2, D3, J2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

Commit message: order new version
Parts:
- added R2: RES-0.0-JUMPER-1/8W-0603, RLC-0603-SMD, symbol RES-0.0-JUMPER-1/8W-0603
Connections:
- net labels removed: BS1, NC1, NC2, NC3, NC4, NC5, NC6, NC7, NC8, VSS
- wire segments 50 -> 54
- no-connect marks 34 -> 33
Other:
- moved on the sheet: J2, Q1, R1

Commit message: added slot and rerouted traces
Parts:
- removed R2: RES-0.0-JUMPER-1/8W-0603, RLC-0603-SMD, symbol RES-0.0-JUMPER-1/8W-0603
- C2: value CAP-CER-1UF -> CAP-CER-2.2UF
Connections:
- net labels removed: TSCL, TSDA
- wire segments 54 -> 51
- no-connect marks 33 -> 36
Changed lines of the file:
@@
 EESchema Schematic File Version 2
-LIBS:wickerlib
+LIBS:kicad-teensy-epaper-rescue
 LIBS:bbd
 LIBS:battery_management
@@
 LIBS:74xx
 LIBS:74xgxx
+LIBS:wickerlib
 LIBS:kicad-teensy-epaper-cache
 EELAYER 25 0
@@
 L HEADER-FEMALE-34POS-FFC-SMT-1x34-P0.5MM J2
 U 1 1 58799DE1
-P 6425 3925
-F 0 "J2" H 6375 4975 50  0000 L CNN
-F 1 "HEADER-FEMALE-34POS-FFC-SMT-1x34-P0.5MM" V 6600 2400 50  0000 L CNN
-F 2 "Wickerlib:CONN-HEADER-FH34SRJ-34S-0.5SH" H 6425 3575 50  0001 C CIN
-F 3 "https://cdn.harwin.com/pdfs/60page140.pd://www.hirose.com/product/en/download_file/key_name/FH34SRJ/category/Catalog/doc_file_id/31646/?file_category_id=4&item_id=27&is_series=1" H 6425 3925 5   0001 C CNN
-F 4 "HEADER FEMALE 34POS SMT 1x34 0.5MMP" H 6425 3575 50  0001 C CIN "Description"
-F 5 "Hirose" H 6425 3575 50  0001 C CIN "MF_Name"
-F 6 "FH34SRJ-34S-0.5SH(99)" H 6425 3575 50  0001 C CIN "MF_PN"
-F 7 "Digikey" H 6425 3575 50  0001 C CIN "S1_Name"
-F 8 "H124726CT-ND" H 6425 3575 50  0001 C CIN "S1_PN"
-	1    6425 3925
-	-1   0    0    1
+P 6425 2525
+F 0 "J2" H 6375 3575 50  0000 L CNN
+F 1 "HEADER-FEMALE-34POS-FFC-SMT-1x34-P0.5MM" V 6600 1000 50  0000 L CNN
+F 2 "Wickerlib:CONN-HEADER-FH34SRJ-34S-0.5SH" H 6425 2175 50  0001 C CIN
+F 3 "https://cdn.harwin.com/pdfs/60page140.pd://www.hirose.com/product/en/download_file/key_name/FH34SRJ/category/Catalog/doc_file_id/31646/?file_category_id=4&item_id=27&is_series=1" H 6425 2525 5   0001 C CNN
+F 4 "HEADER FEMALE 34POS SMT 1x34 0.5MMP" H 6425 2175 50  0001 C CIN "Description"
+F 5 "Hirose" H 6425 2175 50  0001 C CIN "MF_Name"
+F 6 "FH34SRJ-34S-0.5SH(99)" H 6425 2175 50  0001 C CIN "MF_PN"
+F 7 "Digikey" H 6425 2175 50  0001 C CIN "S1_Name"
+F 8 "H124726CT-ND" H 6425 2175 50  0001 C CIN "S1_PN"
+	1    6425 2525
+	-1   0    0    -1
 $EndComp
 Text GLabel 7775 2175 2    50   Input ~ 0
@@
 Text GLabel 7775 2475 2    50   Input ~ 0
 VGH
-Text GLabel 7775 2575 2    50   Input ~ 0
-TSCL
-Text GLabel 7775 2675 2    50   Input ~ 0
-TSDA
 Text GLabel 7775 2875 2    50   Input ~ 0
 BUSY
@@
 VCOM
 $Comp
-L GND #PWR10
+L GND #PWR01
 U 1 1 5893E9A4
 P 8175 2775
-F 0 "#PWR10" H 8175 2525 50  0001 C CNN
+F 0 "#PWR01" H 8175 2525 50  0001 C CNN
 F 1 "GND" H 8175 2625 50  0000 C CNN
 F 2 "" H 8175 2775 50  0000 C CNN
@@
 P 2050 3750
 F 0 "C2" V 2200 3750 50  0000 L CNN
-F 1 "CAP-CER-1UF" V 1925 3475 50  0000 L CNN
+F 1 "CAP-CER-2.2UF" V 1925 3475 50  0000 L CNN
 F 2 "Capacitors_SMD:C_0805_HandSoldering" H 2050 3400 50  0001 C CIN
 F 3 "http://ds.yuden.co.jp/TYCOMPAS/ut/detail.do?productNo=TMK107B7105KA-T&fileName=TMK107B7105KA-T_SS&mode=specSheetDownload" H 2050 3750 5   0001 C CNN
@@
 $EndComp
 $Comp
-L GND #PWR12
+L GND #PWR02
 U 1 1 58941B65
 P 9400 1700
-F 0 "#PWR12" H 9400 1450 50  0001 C CNN
+F 0 "#PWR02" H 9400 1450 50  0001 C CNN
 F 1 "GND" H 9400 1550 50  0000 C CNN
 F 2 "" H 9400 1700 50  0000 C CNN
@@
 $EndComp
 $Comp
-L GND #PWR16
+L GND #PWR03
 U 1 1 58941CF9
 P 9400 3850
-F 0 "#PWR16" H 9400 3600 50  0001 C CNN
+F 0 "#PWR03" H 9400 3600 50  0001 C CNN
 F 1 "GND" H 9400 3700 50  0000 C CNN
 F 2 "" H 9400 3850 50  0000 C CNN
@@
 $EndComp
 $Comp
-L GND #PWR2
+L GND #PWR04
 U 1 1 58941E39
 P 2050 4550
-F 0 "#PWR2" H 2050 4300 50  0001 C CNN
+F 0 "#PWR04" H 2050 4300 50  0001 C CNN
 F 1 "GND" H 2050 4400 50  0000 C CNN
 F 2 "" H 2050 4550 50  0000 C CNN
@@
 $EndComp
 $Comp
-L GND #PWR1
+L GND #PWR05
 U 1 1 58941E7A
 P 1225 3850
-F 0 "#PWR1" H 1225 3600 50  0001 C CNN
+F 0 "#PWR05" H 1225 3600 50  0001 C CNN
 F 1 "GND" H 1225 3700 50  0000 C CNN
 F 2 "" H 1225 3850 50  0000 C CNN
@@
 $EndComp
 $Comp
-L GND #PWR5
+L GND #PWR06
 U 1 1 58941EFC
 P 2950 2950
-F 0 "#PWR5" H 2950 2700 50  0001 C CNN
+F 0 "#PWR06" H 2950 2700 50  0001 C CNN
 F 1 "GND" H 2950 2800 50  0000 C CNN
 F 2 "" H 2950 2950 50  0000 C CNN
@@
 	6625 4875 7775 4875
 Wire Wire Line
-	6625 4775 8000 4775
-Wire Wire Line
 	6625 4675 7775 4675
 Wire Wire Line
@@
 Connection ~ 1225 3275
 $Comp
-L GND #PWR13
+L GND #PWR07
 U 1 1 58952731
 P 9400 2150
-F 0 "#PWR13" H 9400 1900 50  0001 C CNN
+F 0 "#PWR07" H 9400 1900 50  0001 C CNN
 F 1 "GND" H 9400 2000 50  0000 C CNN
 F 2 "" H 9400 2150 50  0000 C CNN
@@
 $EndComp
 $Comp
-L GND #PWR6
+L GND #PWR08
 U 1 1 58953BD1
 P 5050 4625
-F 0 "#PWR6" H 5050 4375 50  0001 C CNN
+F 0 "#PWR08" H 5050 4375 50  0001 C CNN
 F 1 "GND" V 5050 4425 50  0000 C CNN
 F 2 "" H 5050 4625 50  0000 C CNN
@@
 $EndComp
 $Comp
-L GND #PWR15
+L GND #PWR09
 U 1 1 58953E27
 P 9400 2975
-F 0 "#PWR15" H 9400 2725 50  0001 C CNN
+F 0 "#PWR09" H 9400 2725 50  0001 C CNN
 F 1 "GND" H 9400 2825 50  0000 C CNN
 F 2 "" H 9400 2975 50  0000 C CNN
@@
 $EndComp
 $Comp
-L GND #PWR4
+L GND #PWR010
 U 1 1 58954CBF
 P 2900 4625
-F 0 "#PWR4" H 2900 4375 50  0001 C CNN
+F 0 "#PWR010" H 2900 4375 50  0001 C CNN
 F 1 "GND" H 2900 4475 50  0000 C CNN
 F 2 "" H 2900 4625 50  0000 C CNN
@@
 $EndComp
 $Comp
-L GND #PWR14
+L GND #PWR011
 U 1 1 58954E61
 P 9400 2575
-F 0 "#PWR14" H 9400 2325 50  0001 C CNN
+F 0 "#PWR011" H 9400 2325 50  0001 C CNN
 F 1 "GND" V 9400 2375 50  0000 C CNN
 F 2 "" H 9400 2575 50  0000 C CNN
@@
 $EndComp
 $Comp
-L GND #PWR3
+L GND #PWR012
 U 1 1 58955108
 P 2900 3850
-F 0 "#PWR3" H 2900 3600 50  0001 C CNN
+F 0 "#PWR012" H 2900 3600 50  0001 C CNN
 F 1 "GND" V 2900 3650 50  0000 C CNN
 F 2 "" H 2900 3850 50  0000 C CNN
@@
 VSL
 $Comp
-L GND #PWR11
+L GND #PWR013
 U 1 1 589557C5
 P 9375 3350
-F 0 "#PWR11" H 9375 3100 50  0001 C CNN
+F 0 "#PWR013" H 9375 3100 50  0001 C CNN
 F 1 "GND" V 9375 3150 50  0000 C CNN
 F 2 "" H 9375 3350 50  0000 C CNN
@@
 $EndComp
 $Comp
-L GND #PWR8
+L GND #PWR014
 U 1 1 58956AE7
 P 5050 4825
-F 0 "#PWR8" H 5050 4575 50  0001 C CNN
+F 0 "#PWR014" H 5050 4575 50  0001 C CNN
 F 1 "GND" V 5050 4625 50  0000 C CNN
 F 2 "" H 5050 4825 50  0000 C CNN
@@
 $EndComp
 $Comp
-L GND #PWR7
+L GND #PWR015
 U 1 1 58956B28
 P 5050 4725
-F 0 "#PWR7" H 5050 4475 50  0001 C CNN
+F 0 "#PWR015" H 5050 4475 50  0001 C CNN
 F 1 "GND" V 5050 4525 50  0000 C CNN
 F 2 "" H 5050 4725 50  0000 C CNN
@@
 NoConn ~ 7775 4875
 $Comp
-L GND #PWR9
+L GND #PWR016
 U 1 1 58DB75A7
 P 8150 3675
-F 0 "#PWR9" H 8150 3425 50  0001 C CNN
+F 0 "#PWR016" H 8150 3425 50  0001 C CNN
 F 1 "GND" H 8150 3525 50  0000 C CNN
 F 2 "" H 8150 3675 50  0000 C CNN
@@
 	0    -1   -1   0
 $EndComp
-$Comp
-L RES-0.0-JUMPER-1/8W-0603 R2
-U 1 1 58DB7A3A
-P 8450 4800
-F 0 "R2" H 8500 4850 50  0000 L CNN
-F 1 "RES-0.0-JUMPER-1/8W-0603" H 8500 4750 50  0000 L CNN
-F 2 "RLC-0603-SMD" H 8450 4450 50  0001 C CIN
-F 3 "http://www.vishay.com/docs/28705/mcx0x0xpro.pdf" H 8450 4800 5   0001 C CNN
-F 4 "RES SMD 0.0 OHM JUMPER 1/8W 0603" H 8450 4450 50  0001 C CIN "Description"
-F 5 "Vishay" H 8450 4450 50  0001 C CIN "MF_Name"
-F 6 "MCT06030Z0000ZP500" H 8450 4450 50  0001 C CIN "MF_PN"
-F 7 "Digikey" H 8450 4450 50  0001 C CIN "S1_Name"
-F 8 "MCT0603-0.0-ZZCT-ND" H 8450 4450 50  0001 C CIN "S1_PN"
-	1    8450 4800
-	1    0    0    -1
-$EndComp
-Wire Wire Line
-	8000 4700 8000 4900
-Wire Wire Line
-	8000 4700 8450 4700
-Wire Wire Line
-	8000 4900 8450 4900
-Connection ~ 8000 4775
+Wire Wire Line
+	6625 4775 7775 4775
+NoConn ~ 7775 4775
+NoConn ~ 7775 2575
+NoConn ~ 7775 2675
 $EndSCHEMATC
